Commit message: add random camera to test position

File: src/niryo_one_description/urdf/niryo_one.urdf.xacro (robot description, xacro)
@@ -503,3 +503,69 @@
     </joint>
     <!-- Adding RealSense Sensor  -->
+    <joint name="camera_joint" type="fixed">
+        <axis xyz="0 0 0" />
+        <origin xyz="0.18644192 0.17179403 0.29468409" rpy="-2.5516856 -0.9516703 -2.0573373"/>
+        <parent link="base_link"/>
+        <child link="camera_link"/>
+    </joint>
+      <!-- Camera -->
+    <link name="camera_link">
+        <collision>
+        <origin xyz="0 0 0" rpy="0 0 0"/>
+        <geometry>
+        <box size="0.05 0.05 0.05"/>
+        </geometry>
+        </collision>
+        <visual>
+        <origin xyz="0 0 0" rpy="0 0 0"/>
+        <geometry>
+        <box size="0.05 0.05 0.05"/>
+        </geometry>
+        <material name="red"/>
+        </visual>
+        <inertial>
+        <mass value="1e-5" />
+        <origin xyz="0 0 0.0" rpy="0 0 0"/>
+        <inertia ixx="1e-6" ixy="0" ixz="0" iyy="1e-6" iyz="0" izz="1e-6" />
+        </inertial>
+    </link>
+    <gazebo reference="camera_link">
+        <sensor type="camera" name="camera1">
+        <update_rate>30.0</update_rate>
+        <camera name="head">
+            <horizontal_fov>1.3962634</horizontal_fov>
+            <image>
+            <width>800</width>
+            <height>800</height>
+            <format>R8G8B8</format>
+            </image>
+            <clip>
+            <near>0.02</near>
+            <far>300</far>
+            </clip>
+            <noise>
+            <type>gaussian</type>
+            <!-- Noise is sampled independently per pixel on each frame.
+                That pixel's noise value is added to each of its color
+                channels, which at that point lie in the range [0,1]. -->
+            <mean>0.0</mean>
+            <stddev>0.007</stddev>
+            </noise>
+        </camera>
+        <plugin name="camera_controller" filename="libgazebo_ros_camera.so">
+            <alwaysOn>true</alwaysOn>
+            <updateRate>0.0</updateRate>
+            <cameraName>niryo/camera1</cameraName>
+            <imageTopicName>image_raw</imageTopicName>
+            <cameraInfoTopicName>camera_info</cameraInfoTopicName>
+            <frameName>camera_link</frameName>
+            <hackBaseline>0.07</hackBaseline>
+            <distortionK1>0.0</distortionK1>
+            <distortionK2>0.0</distortionK2>
+            <distortionK3>0.0</distortionK3>
+            <distortionT1>0.0</distortionT1>
+            <distortionT2>0.0</distortionT2>
+        </plugin>
+        </sensor>
+    </gazebo>
 </robot>

Commit message: Update niryo_one.urdf.xacro

File: src/niryo_one_description/urdf/niryo_one.urdf.xacro (robot description, xacro)
@@ -505,5 +505,5 @@
     <joint name="camera_joint" type="fixed">
         <axis xyz="0 0 0" />
-        <origin xyz="0.18644192 0.17179403 0.29468409" rpy="-2.5516856 -0.9516703 -2.0573373"/>
+        <origin xyz="-0.101 0.274 0.257" rpy="-2.083 -0.176 -1.850"/>
         <parent link="base_link"/>
         <child link="camera_link"/>

Commit message: modify the model, camera now working well (still not intel)

File: src/niryo_one_description/urdf/niryo_one.urdf.xacro (robot description, xacro)
@@ -504,5 +504,5 @@
     <!-- Adding RealSense Sensor  -->
     <joint name="camera_joint" type="fixed">
-        <axis xyz="0 0 0" />
+        <axis xyz="0 1 0" />
         <origin xyz="-0.101 0.274 0.257" rpy="-2.083 -0.176 -1.850"/>
         <parent link="base_link"/>
@@ -530,5 +530,14 @@
         </inertial>
     </link>
-    <gazebo reference="camera_link">
+    <!-- Camera Adujustment (it's originally set to point in x, gotta rotate around y by 90) -->
+    <joint name="camera_joint_fix" type="fixed">
+        <axis xyz="0 1 0" />
+        <origin xyz="0 0 0" rpy="0 -1.5 1.5"/>
+        <parent link="camera_link"/>
+        <child link="camera_link_adjust"/>
+    </joint>
+    <link name="camera_link_adjust">
+    </link>
+    <gazebo reference="camera_link_adjust">
         <sensor type="camera" name="camera1">
         <update_rate>30.0</update_rate>
@@ -536,6 +545,6 @@
             <horizontal_fov>1.3962634</horizontal_fov>
             <image>
-            <width>800</width>
-            <height>800</height>
+            <width>1920</width>
+            <height>1080</height>
             <format>R8G8B8</format>
             </image>
